File: pcb/Trabajo_Practico/Trabajo_Practico.sch (KiCad schematic (older format))
At the start: 13 parts, among them J1 Conn_02x19_Odd_Even, J2 Conn_02x19_Odd_Even, J3 Conn_01x03_Male, J4 Conn_01x03_Male, U1 ESP8266-01_ESP-01, U2 MAX30102_P, U3 SD_Card_P, U4 DS18B20

Commit message: Se agrega el Power Flag
Parts:
- added H1, H2, H3, H4: MountingHole, symbol Mechanical:MountingHole
Connections:
- net labels added: 3.3V_STM32
- wire segments 144 -> 150
- no-connect marks 30 -> 79
Other:
- note added: "PWR_FLAG GND"
- note added: "PWR_FLAG VCC"
- moved on the sheet: J3, J4

Commit message: Se ordena los componentes en el pcb
Parts:
- H1, H2, H3, H4: footprint (none) -> MountingHole:MountingHole_2.2mm_M2_Pad_Via
Changed lines of the file:
@@
 F 0 "H1" H 5600 4296 50  0000 L CNN
 F 1 "MountingHole" H 5600 4205 50  0000 L CNN
-F 2 "" H 5500 4250 50  0001 C CNN
+F 2 "MountingHole:MountingHole_2.2mm_M2_Pad_Via" H 5500 4250 50  0001 C CNN
 F 3 "~" H 5500 4250 50  0001 C CNN
 	1    5500 4250
@@
 F 0 "H3" H 6400 4296 50  0000 L CNN
 F 1 "MountingHole" H 6400 4205 50  0000 L CNN
-F 2 "" H 6300 4250 50  0001 C CNN
+F 2 "MountingHole:MountingHole_2.2mm_M2_Pad_Via" H 6300 4250 50  0001 C CNN
 F 3 "~" H 6300 4250 50  0001 C CNN
 	1    6300 4250
@@
 F 0 "H2" H 5600 4696 50  0000 L CNN
 F 1 "MountingHole" H 5600 4605 50  0000 L CNN
-F 2 "" H 5500 4650 50  0001 C CNN
+F 2 "MountingHole:MountingHole_2.2mm_M2_Pad_Via" H 5500 4650 50  0001 C CNN
 F 3 "~" H 5500 4650 50  0001 C CNN
 	1    5500 4650
@@
 F 0 "H4" H 6400 4696 50  0000 L CNN
 F 1 "MountingHole" H 6400 4605 50  0000 L CNN
-F 2 "" H 6300 4650 50  0001 C CNN
+F 2 "MountingHole:MountingHole_2.2mm_M2_Pad_Via" H 6300 4650 50  0001 C CNN
 F 3 "~" H 6300 4650 50  0001 C CNN
 	1    6300 4650

Commit message: Se realizaron las correcciones
Parts:
- U4: footprint Package_TO_SOT_THT:TO-92_Inline -> Connector_PinHeader_2.54mm:PinHeader_1x03_P2.54mm_Vertical
- renumbered U3 to J5
Connections:
- net labels removed: 3.3V_STM32
- wire segments 150 -> 149
Other:
- note added: "PWR_FLAG \nGND"
- note added: "VCC 3.3v"
- note removed: "PWR_FLAG GND"
- moved on the sheet: H1, H2, H3, H4
Changed lines of the file:
@@
 encoding utf-8
 Sheet 1 1
-Title "Ing. Williams Ernesto Limonchi Sandoval"
+Title "Módulo Detector de Caídas para STM32"
 Date "2021-07-02"
 Rev "V1.0"
-Comp "Módulo Detector de Caídas para STM32"
+Comp "Ing. William's Ernesto Limonchi Sandoval"
 Comment1 "Basado en: https://bit.ly/37dJ0iX"
 Comment2 "Revisor 1: Ing. German Cardozo"
@@
 L power:GND #PWR01
 U 1 1 6112A276
-P 1350 2450
-F 0 "#PWR01" H 1350 2200 50  0001 C CNN
-F 1 "GND" H 1355 2277 50  0000 C CNN
-F 2 "" H 1350 2450 50  0001 C CNN
-F 3 "" H 1350 2450 50  0001 C CNN
-	1    1350 2450
+P 1200 2450
+F 0 "#PWR01" H 1200 2200 50  0001 C CNN
+F 1 "GND" H 1205 2277 50  0000 C CNN
+F 2 "" H 1200 2450 50  0001 C CNN
+F 3 "" H 1200 2450 50  0001 C CNN
+	1    1200 2450
 	-1   0    0    -1
 $EndComp
@@
 	1900 2500 1700 2500
 Wire Wire Line
-	1900 2300 1350 2300
-Wire Wire Line
-	1350 2300 1350 2450
-Wire Wire Line
 	2600 1400 2400 1400
 Wire Wire Line
@@
 $EndComp
 $Comp
-L SD_Card:SD_Card_P U3
+L SD_Card:SD_Card_P J5
 U 1 1 611439E4
 P 9300 5400
-F 0 "U3" H 10378 5223 79  0000 L CNN
+F 0 "J5" H 10378 5223 79  0000 L CNN
 F 1 "SD_Card_P" H 10378 5088 79  0000 L CNN
 F 2 "TP_Footprints:SD_CARD_P" H 9600 5700 79  0001 C CNN
@@
 F 0 "U4" H 9570 4046 50  0000 R CNN
 F 1 "DS18B20" H 9570 3955 50  0000 R CNN
-F 2 "Package_TO_SOT_THT:TO-92_Inline" H 8800 3750 50  0001 C CNN
+F 2 "Connector_PinHeader_2.54mm:PinHeader_1x03_P2.54mm_Vertical" H 8800 3750 50  0001 C CNN
 F 3 "http://datasheets.maximintegrated.com/en/ds/DS18B20.pdf" H 9650 4250 50  0001 C CNN
 	1    9800 4000
@@
 	10000 1300 10000 1200
 $Comp
-L power:VCC #PWR0105
-U 1 1 614AFDC9
-P 4750 4450
-F 0 "#PWR0105" H 4750 4300 50  0001 C CNN
-F 1 "VCC" H 4765 4623 50  0000 C CNN
-F 2 "" H 4750 4450 50  0001 C CNN
-F 3 "" H 4750 4450 50  0001 C CNN
-	1    4750 4450
-	1    0    0    -1
-$EndComp
-Text Label 2600 2100 0    47   ~ 0
-3.3V_STM32
-$Comp
-L power:PWR_FLAG #FLG0101
-U 1 1 614B99E2
-P 5050 4450
-F 0 "#FLG0101" H 5050 4525 50  0001 C CNN
-F 1 "PWR_FLAG" H 5050 4600 50  0000 C CNN
-F 2 "" H 5050 4450 50  0001 C CNN
-F 3 "~" H 5050 4450 50  0001 C CNN
-	1    5050 4450
-	1    0    0    -1
-$EndComp
-$Comp
 L power:GND #PWR0106
 U 1 1 614E42FA
-P 3300 2400
-F 0 "#PWR0106" H 3300 2150 50  0001 C CNN
-F 1 "GND" H 3305 2227 50  0000 C CNN
-F 2 "" H 3300 2400 50  0001 C CNN
-F 3 "" H 3300 2400 50  0001 C CNN
-	1    3300 2400
+P 3200 2450
+F 0 "#PWR0106" H 3200 2200 50  0001 C CNN
+F 1 "GND" H 3205 2277 50  0000 C CNN
+F 2 "" H 3200 2450 50  0001 C CNN
+F 3 "" H 3200 2450 50  0001 C CNN
+	1    3200 2450
 	1    0    0    -1
 $EndComp
@@
 L power:PWR_FLAG #FLG0102
 U 1 1 614ED268
-P 3300 2300
-F 0 "#FLG0102" H 3300 2375 50  0001 C CNN
-F 1 "PWR_FLAG" H 3300 2450 50  0000 C CNN
-F 2 "" H 3300 2300 50  0001 C CNN
-F 3 "~" H 3300 2300 50  0001 C CNN
-	1    3300 2300
-	1    0    0    -1
-$EndComp
-Text Label 4650 4650 2    79   ~ 0
-3.3V_STM32
-Wire Wire Line
-	4750 4450 4900 4450
-Wire Wire Line
-	4650 4650 4900 4650
-Wire Wire Line
-	4900 4650 4900 4450
-Connection ~ 4900 4450
-Wire Wire Line
-	4900 4450 5050 4450
-Wire Notes Line
-	5300 4000 5300 4950
+P 1200 2250
+F 0 "#FLG0102" H 1200 2325 50  0001 C CNN
+F 1 "PWR_FLAG" H 1200 2400 50  0000 C CNN
+F 2 "" H 1200 2250 50  0001 C CNN
+F 3 "~" H 1200 2250 50  0001 C CNN
+	1    1200 2250
+	1    0    0    -1
+$EndComp
 Wire Wire Line
 	2850 2300 2850 2350
-Wire Wire Line
-	3300 2350 2850 2350
 Connection ~ 2850 2350
 Wire Wire Line
 	2850 2350 2850 2400
-Wire Wire Line
-	3300 2350 3300 2300
-Wire Wire Line
-	3300 2400 3300 2350
-Connection ~ 3300 2350
-Text Notes 4500 4200 2    59   ~ 0
+Text Notes 3650 2250 2    59   ~ 0
 PWR_FLAG VCC
-Text Notes 3650 3150 2    59   ~ 0
-PWR_FLAG GND
-Wire Notes Line
-	3300 3200 3700 3200
-Wire Notes Line
-	3700 3200 3700 3000
-Wire Notes Line
-	3700 3000 3500 3000
-Wire Notes Line
-	3500 3000 3500 2350
-Wire Notes Line
-	3500 2350 3400 2350
-Wire Wire Line
-	2600 2100 2400 2100
+Text Notes 650  2400 0    59   ~ 0
+PWR_FLAG \nGND
 Wire Notes Line
 	6500 3800 6850 3800
@@
 L Mechanical:MountingHole H1
 U 1 1 61586865
-P 5500 4250
-F 0 "H1" H 5600 4296 50  0000 L CNN
-F 1 "MountingHole" H 5600 4205 50  0000 L CNN
-F 2 "MountingHole:MountingHole_2.2mm_M2_Pad_Via" H 5500 4250 50  0001 C CNN
-F 3 "~" H 5500 4250 50  0001 C CNN
-	1    5500 4250
+P 4750 4250
+F 0 "H1" H 4850 4296 50  0000 L CNN
+F 1 "MountingHole" H 4850 4205 50  0000 L CNN
+F 2 "MountingHole:MountingHole_2.2mm_M2_Pad_Via" H 4750 4250 50  0001 C CNN
+F 3 "~" H 4750 4250 50  0001 C CNN
+	1    4750 4250
 	1    0    0    -1
 $EndComp
@@
 L Mechanical:MountingHole H3
 U 1 1 615876E8
-P 6300 4250
-F 0 "H3" H 6400 4296 50  0000 L CNN
-F 1 "MountingHole" H 6400 4205 50  0000 L CNN
-F 2 "MountingHole:MountingHole_2.2mm_M2_Pad_Via" H 6300 4250 50  0001 C CNN
-F 3 "~" H 6300 4250 50  0001 C CNN
-	1    6300 4250
+P 5550 4250
+F 0 "H3" H 5650 4296 50  0000 L CNN
+F 1 "MountingHole" H 5650 4205 50  0000 L CNN
+F 2 "MountingHole:MountingHole_2.2mm_M2_Pad_Via" H 5550 4250 50  0001 C CNN
+F 3 "~" H 5550 4250 50  0001 C CNN
+	1    5550 4250
 	1    0    0    -1
 $EndComp
@@
 L Mechanical:MountingHole H2
 U 1 1 61587E15
-P 5500 4650
-F 0 "H2" H 5600 4696 50  0000 L CNN
-F 1 "MountingHole" H 5600 4605 50  0000 L CNN
-F 2 "MountingHole:MountingHole_2.2mm_M2_Pad_Via" H 5500 4650 50  0001 C CNN
-F 3 "~" H 5500 4650 50  0001 C CNN
-	1    5500 4650
+P 4750 4650
+F 0 "H2" H 4850 4696 50  0000 L CNN
+F 1 "MountingHole" H 4850 4605 50  0000 L CNN
+F 2 "MountingHole:MountingHole_2.2mm_M2_Pad_Via" H 4750 4650 50  0001 C CNN
+F 3 "~" H 4750 4650 50  0001 C CNN
+	1    4750 4650
 	1    0    0    -1
 $EndComp
@@
 L Mechanical:MountingHole H4
 U 1 1 61588339
-P 6300 4650
-F 0 "H4" H 6400 4696 50  0000 L CNN
-F 1 "MountingHole" H 6400 4605 50  0000 L CNN
-F 2 "MountingHole:MountingHole_2.2mm_M2_Pad_Via" H 6300 4650 50  0001 C CNN
-F 3 "~" H 6300 4650 50  0001 C CNN
-	1    6300 4650
-	1    0    0    -1
-$EndComp
+P 5550 4650
+F 0 "H4" H 5650 4696 50  0000 L CNN
+F 1 "MountingHole" H 5650 4605 50  0000 L CNN
+F 2 "MountingHole:MountingHole_2.2mm_M2_Pad_Via" H 5550 4650 50  0001 C CNN
+F 3 "~" H 5550 4650 50  0001 C CNN
+	1    5550 4650
+	1    0    0    -1
+$EndComp
+Wire Wire Line
+	3200 2450 3200 2350
+Wire Wire Line
+	3200 2350 2850 2350
+Wire Wire Line
+	3100 2100 3100 1950
+Wire Wire Line
+	2400 2100 3100 2100
+$Comp
+L power:VCC #PWR0105
+U 1 1 611720F7
+P 3100 1950
+F 0 "#PWR0105" H 3100 1800 50  0001 C CNN
+F 1 "VCC" H 3115 2123 50  0000 C CNN
+F 2 "" H 3100 1950 50  0001 C CNN
+F 3 "" H 3100 1950 50  0001 C CNN
+	1    3100 1950
+	1    0    0    -1
+$EndComp
+Text Notes 3050 1700 0    79   ~ 0
+VCC 3.3v
+Wire Wire Line
+	1200 2250 1200 2300
+$Comp
+L power:PWR_FLAG #FLG0101
+U 1 1 61183451
+P 3400 2050
+F 0 "#FLG0101" H 3400 2125 50  0001 C CNN
+F 1 "PWR_FLAG" H 3400 2200 50  0000 C CNN
+F 2 "" H 3400 2050 50  0001 C CNN
+F 3 "~" H 3400 2050 50  0001 C CNN
+	1    3400 2050
+	1    0    0    -1
+$EndComp
+Wire Wire Line
+	3400 2050 3400 2100
+Wire Wire Line
+	3400 2100 3100 2100
+Connection ~ 3100 2100
+Wire Wire Line
+	1200 2300 1900 2300
+Wire Wire Line
+	1200 2450 1200 2300
+Connection ~ 1200 2300
 $EndSCHEMATC

Commit message: Presentacion final del proyecto
Parts:
- added C4: 100nF, Capacitor_SMD:C_0805_2012Metric, symbol Device:C
- added D1: LED, LED_SMD:LED_0805_2012Metric_Pad1.15x1.40mm_HandSolder, symbol Device:LED
- added FID1, FID2, FID3, FID4: Fiducial, Fiducial:Fiducial_0.5mm_Mask1mm, symbol Mechanical:Fiducial
- added R2: 330, Resistor_SMD:R_0805_2012Metric, symbol Device:R
- U2: symbol max30102:MAX30102_P -> Trabajo_Practico-rescue:MAX30102_P-max30102
Connections:
- wire segments 149 -> 166
Other:
- note added: "LED indicador\nde alimentación"
- moved on the sheet: C1, C2, C3, H1, H2, H3, H4, J3, J4, J5, U4

Commit message: Agrego sensor MLX90614
Parts:
- removed U1: ESP8266-01_ESP-01, TP_Footprints:ESP-01, symbol ESP8266-01_ESP-01:ESP8266-01_ESP-01
- removed U4: DS18B20, Connector_PinHeader_2.54mm:PinHeader_1x03_P2.54mm_Vertical, symbol Sensor_Temperature:DS18B20
- added J6: Conn_01x02_Female, Connector_PinSocket_2.54mm:PinSocket_1x02_P2.54mm_Vertical, symbol Connector:Conn_01x02_Female
- added R3: 10k, Resistor_SMD:R_0805_2012Metric, symbol Device:R
- added R4: 1k, Resistor_SMD:R_0805_2012Metric, symbol Device:R
- added U1: Tiny_Fox, TP_Footprints:TinyFox, symbol Trabajo_Practico-rescue:Tiny_Fox
- added U3: MLX90614, TP_Footprints:MLX90614, symbol Trabajo_Practico-rescue:MLX90614
- R1: value 10k -> 1k
- U2: value MAX30102_P -> MAX30102_P-max30102
Connections:
- net AN0 is gone; now on net PC15: J1.28 (Pin_28)
- net PA1 is gone; now on net PH0: J1.30 (Pin_30)
- net PA4 is gone; now on net PH1: J1.32 (Pin_32)
- net +5V: now also J1.17 (Pin_17), U3.4 (VCC); no longer J1.18 (Pin_18)
- net AGND: now also J2.31 (Pin_31); no longer J2.32 (Pin_32)
- net AVDD: now also J2.8 (Pin_8); no longer J2.7 (Pin_7)
- net BOT0: now also J1.8 (Pin_8); no longer J1.7 (Pin_7)
- net CLK: now also J2.26 (Pin_26); no longer J2.25 (Pin_25)
- net CS: now also J2.18 (Pin_18); no longer J2.17 (Pin_17)
- net E5V: now also J1.5 (Pin_5); no longer J1.6 (Pin_6)
- net GND: now also J1.21 (Pin_21), J1.7 (Pin_7), J2.10 (Pin_10), J2.19 (Pin_19), U2.2 (GND), J6.1 (Pin_1), U1.1 (G), U1.6 (G), U3.3 (GND); no longer J1.22 (Pin_22), J1.8 (Pin_8), J2.20 (Pin_20), J2.9 (Pin_9)
- net IOREF: now also J1.11 (Pin_11); no longer J1.12 (Pin_12)
- net MISO: now also J1.36 (Pin_36), J5.15 (MISO); no longer J1.35 (Pin_35), J5.7 (MISO)
- net MOSI: now also J1.38 (Pin_38), J5.13 (MOSI); no longer J1.37 (Pin_37), J5.5 (MOSI)
- net PA10: now also J2.34 (Pin_34), U1.3 (TX); no longer J2.33 (Pin_33)
- net PA11: now also J2.13 (Pin_13); no longer J2.14 (Pin_14)
- net PA12: now also J2.11 (Pin_11); no longer J2.12 (Pin_12)
- net PA13: now also J1.14 (Pin_14); no longer J1.13 (Pin_13)
- net PA14: now also J1.16 (Pin_16); no longer J1.15 (Pin_15)
- net PA15: now also J1.18 (Pin_18); no longer J1.17 (Pin_17)
- net PA2: now also J2.36 (Pin_36); no longer J2.35 (Pin_35)
- net PA3: now also J2.38 (Pin_38); no longer J2.37 (Pin_37)
- net PA5: now also J2.12 (Pin_12); no longer J2.11 (Pin_11)
- net PA6: now also J2.14 (Pin_14); no longer J2.13 (Pin_13)
- net PA7: now also J2.16 (Pin_16); no longer J2.15 (Pin_15)
- net PA8: now also J2.24 (Pin_24); no longer J2.23 (Pin_23)
- net PA9: now also J2.22 (Pin_22), U1.2 (RX); no longer J2.21 (Pin_21)
- net PB0: now also J1.33 (Pin_33); no longer J1.34 (Pin_34)
- net PB1: now also J2.23 (Pin_23); no longer J2.24 (Pin_24)
- net PB12: now also J2.15 (Pin_15); no longer J2.16 (Pin_16)
- net PB13: now also J2.29 (Pin_29); no longer J2.30 (Pin_30)
- net PB14: now also J2.27 (Pin_27); no longer J2.28 (Pin_28)
- net PB15: now also J2.25 (Pin_25); no longer J2.26 (Pin_26)
- net PB2: now also J2.21 (Pin_21); no longer J2.22 (Pin_22)
- net PB3: now also J2.32 (Pin_32); no longer J2.31 (Pin_31)
- net PB4: now also J2.28 (Pin_28); no longer J2.27 (Pin_27)
- net PB5: now also J2.30 (Pin_30); no longer J2.29 (Pin_29)
- net PB7: now also J1.22 (Pin_22); no longer J1.21 (Pin_21)
- net PB8: now also J2.4 (Pin_4), U2.3 (SCL), U3.2 (SCL); no longer J2.3 (Pin_3)
- net PB9: now also J2.6 (Pin_6), U2.4 (SDA), U3.1 (SDA); no longer J2.5 (Pin_5)
- net PC0: now also J1.37 (Pin_37), U2.5 (INT), R3.2; no longer J1.38 (Pin_38)
- net PC1: now also J1.35 (Pin_35); no longer J1.36 (Pin_36)
- net PC10: now also J1.2 (Pin_2); no longer J1.1 (Pin_1)
- net PC11: now also J1.1 (Pin_1); no longer J1.2 (Pin_2)
- net PC12: now also J1.4 (Pin_4); no longer J1.3 (Pin_3)
- net PC13: now also J1.24 (Pin_24); no longer J1.23 (Pin_23)
- net PC14: now also J1.26 (Pin_26); no longer J1.25 (Pin_25)
- net PC15: no longer J1.27 (Pin_27)
- net PC4: now also J2.33 (Pin_33); no longer J2.34 (Pin_34)
- net PC5: now also J2.5 (Pin_5); no longer J2.6 (Pin_6)
- net PC6: now also J2.3 (Pin_3); no longer J2.4 (Pin_4)
- net PC7: now also J2.20 (Pin_20); no longer J2.19 (Pin_19)
- net PC8: now also J2.1 (Pin_1); no longer J2.2 (Pin_2)
- net PC9: now also J2.2 (Pin_2); no longer J2.1 (Pin_1)
- net PD2: now also J1.3 (Pin_3); no longer J1.4 (Pin_4)
- net PH0: no longer J1.29 (Pin_29)
- net PH1: no longer J1.31 (Pin_31)
- net RESET: now also J1.13 (Pin_13); no longer J1.14 (Pin_14)
- net U5V: now also J2.7 (Pin_7); no longer J2.8 (Pin_8)
- net VBAT: now also J1.34 (Pin_34); no longer J1.33 (Pin_33)
- net VCC: now also J1.15 (Pin_15), U2.1 (VIN), R3.1, U1.5 (3.3V); no longer J1.16 (Pin_16), R1.2
- net VDD: now also J1.6 (Pin_6); no longer J1.5 (Pin_5)
- net VIN: now also J1.23 (Pin_23); no longer J1.24 (Pin_24)
- net AN1: now reaches R1.1
- net AN1: now also J1.29 (Pin_29), R4.2
- new net: J6.2 (Pin_2), R1.2
- new net M_BAT: J1.31 (Pin_31), R4.1
- new net PA0: J1.27 (Pin_27)
- no-connect marks 79 -> 68
Other:
- note added: "MODULO SIGFOX\nTINYFOX"
- note added: "Medidor Bateria"
- note added: "Para la comunicación \nse utiliza el módulo\nTinyFox de Teca"
- note removed: "MODULO WIFI\nESP8266-01"
- note removed: "Para este caso no \nse usan los GPIOs"
- moved on the sheet: C1, C2, C3, FID1, FID2, FID3, FID4, H1, H2, H3, H4
